File: boards/roomnode-s3/roomnode-s3.kicad_sch (KiCad schematic)
At the start: 11 parts, among them J1 USB-C TYPE-C-31-M-12, J2 HLK-LD2450, J3 AM312 PIR, SW1 EN, SW2 BOOT, U1 ESP32-S3-WROOM-1-N8R2, U2 ME6211C33M5G, U3 SHT40, U4 SGP40, U5 BH1750

Commit message: Regenerate roomnode-s3 KiCad design files
Parts:
- added D1: USBLC6-2SC6 ESD, symbol local:Box
- J1: value USB-C TYPE-C-31-M-12 -> USB-C C165948 16p
- SW1: value EN -> EN + R4 10k + C5 100nF
- SW2: value BOOT -> BOOT + R5 10k
- U2: value ME6211C33M5G -> AMS1117-3.3 (C6186)
Other:
- title: RoomNode-S3 rev A -> RoomNode-S3 rev B
